File: powersupplies_kicadproject.kicad_pcb (KiCad board)
At the start: 6 copper layers, 160 x 99 mm, 6 parts

Commit message: Save progress.
Parts:
- added C1: 10uF, Capacitor_SMD:C_1206_3216Metric_Pad1.33x1.80mm_HandSolder, F.Cu at (193.7, 92.4)
- added C2: 10uF, Capacitor_SMD:C_1206_3216Metric_Pad1.33x1.80mm_HandSolder, F.Cu at (193.7, 95.8)
- added C3: 10uF, Capacitor_SMD:C_1206_3216Metric_Pad1.33x1.80mm_HandSolder, F.Cu at (193.7, 99.1)
- added C4: 10uF, Capacitor_SMD:C_1206_3216Metric_Pad1.33x1.80mm_HandSolder, F.Cu at (193.7, 102.5)
- added C5: 10uF, Capacitor_SMD:C_1206_3216Metric_Pad1.33x1.80mm_HandSolder, F.Cu at (193.7, 105.8)
- added C6: 10uF, Capacitor_SMD:C_1206_3216Metric_Pad1.33x1.80mm_HandSolder, F.Cu at (193.7, 109.2)
- added C7: 10uF, Capacitor_SMD:C_1206_3216Metric_Pad1.33x1.80mm_HandSolder, F.Cu at (193.7, 112.5)
- added C8: 10uF, Capacitor_SMD:C_1206_3216Metric_Pad1.33x1.80mm_HandSolder, F.Cu at (193.7, 115.9)
- added F1: Fuse, Fuse:Fuse_Littelfuse-NANO2-451_453, F.Cu at (230.0, 129.2)
- added F2: Fuse, Fuse:Fuse_Littelfuse-NANO2-451_453, F.Cu at (230.0, 73.3)
- added U2: TSR2-2465, Converter_DCDC:Converter_DCDC_TRACO_TSR2-xxxx_THT, F.Cu at (200.0, 129.2)
- added U3: TSR2-2465, Converter_DCDC:Converter_DCDC_TRACO_TSR2-xxxx_THT, F.Cu at (200.0, 73.3)
Connections:
- net /Conn_DIN41612_48pin/+15V renamed /6.5V Dual Rail Power/+15V
- net /Conn_DIN41612_48pin/+6.5V renamed /6.5V Dual Rail Power/+6.5V
- net /Conn_DIN41612_48pin/-15V renamed /6.5V Dual Rail Power/-15V
- net /Conn_DIN41612_48pin/-6.5V renamed /6.5V Dual Rail Power/-6.5V
Routing:
- net /6.5V Dual Rail Power/-6.5V: track 5.08 -> 22.0 mm
- net /6.5V Dual Rail Power/+6.5V: track 5.08 -> 22.0 mm

Commit message: Save progress.
Parts:
- moved C1 40.2 mm to (213.0, 127.6), turned to 90 degrees
- moved C2 39.5 mm to (217.0, 127.6), turned to 90 degrees
- moved C8 36.6 mm to (205.9, 81.4), turned to 90 degrees
- moved C4 36.1 mm to (217.0, 74.9), turned to 90 degrees
- moved C7 32.4 mm to (202.5, 81.4), turned to 90 degrees
- moved C3 31.0 mm to (213.0, 74.9), turned to 90 degrees
- moved C5 22.3 mm to (188.9, 127.6), turned to 90 degrees
- moved C6 18.5 mm to (192.3, 127.6), turned to 90 degrees
Routing:
- net Net-(U3-Vout): track 0.00 -> 22.5 mm
- net Net-(U2-Vout): track 0.00 -> 22.5 mm
- net /6.5V Dual Rail Power/+15V: track 5.08 -> 16.2 mm
- net /6.5V Dual Rail Power/-15V: track 5.08 -> 14.9 mm
