File: Conn_DIN41612_48pin.kicad_sch (KiCad schematic)
At the start: 1 part

Commit message: Save progress.
Changed lines of the file:
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@@
 	)
 	(hierarchical_label "-15V"
-		(shape input)
+		(shape output)
 		(at 133.35 38.1 180)
 		(effects
@@
 	)
 	(hierarchical_label "+15V"
-		(shape input)
+		(shape output)
 		(at 203.2 133.35 180)
 		(effects
@@
 	)
 	(hierarchical_label "+15V"
-		(shape input)
+		(shape output)
 		(at 63.5 133.35 180)
 		(effects
@@
 	)
 	(hierarchical_label "-15V"
-		(shape input)
+		(shape output)
 		(at 203.2 38.1 180)
 		(effects
@@
 	)
 	(hierarchical_label "+15V"
-		(shape input)
+		(shape output)
 		(at 133.35 133.35 180)
 		(effects
@@
 	)
 	(hierarchical_label "-15V"
-		(shape input)
+		(shape output)
 		(at 63.5 38.1 180)
 		(effects
@@
 		)
 		(instances
-			(project "Eurocard_48pin_AMO_Blank"
+			(project "powersupplies_kicadproject"
 				(path "/d2bb73ea-a6bc-4588-b3f4-545ae2e25abc/b247aa19-c6db-40d4-9578-4858bd0a46c8"
 					(reference "#PWR05")
@@
 		)
 		(instances
-			(project "Eurocard_48pin_AMO_Blank"
+			(project "powersupplies_kicadproject"
 				(path "/d2bb73ea-a6bc-4588-b3f4-545ae2e25abc/b247aa19-c6db-40d4-9578-4858bd0a46c8"
 					(reference "#PWR04")
@@
 		)
 		(instances
-			(project "Eurocard_48pin_AMO_Blank"
+			(project "powersupplies_kicadproject"
 				(path "/d2bb73ea-a6bc-4588-b3f4-545ae2e25abc/b247aa19-c6db-40d4-9578-4858bd0a46c8"
 					(reference "#PWR07")
@@
 		)
 		(instances
-			(project "Eurocard_48pin_AMO_Blank"
+			(project "powersupplies_kicadproject"
 				(path "/d2bb73ea-a6bc-4588-b3f4-545ae2e25abc/b247aa19-c6db-40d4-9578-4858bd0a46c8"
 					(reference "#PWR03")
@@
 		)
 		(instances
-			(project "Eurocard_48pin_AMO_Blank"
+			(project "powersupplies_kicadproject"
 				(path "/d2bb73ea-a6bc-4588-b3f4-545ae2e25abc/b247aa19-c6db-40d4-9578-4858bd0a46c8"
 					(reference "#PWR08")
@@
 		)
 		(instances
-			(project "Eurocard_48pin_AMO_Blank"
+			(project "powersupplies_kicadproject"
 				(path "/d2bb73ea-a6bc-4588-b3f4-545ae2e25abc/b247aa19-c6db-40d4-9578-4858bd0a46c8"
 					(reference "#PWR09")
@@
 		)
 		(instances
-			(project "Eurocard_48pin_AMO_Blank"
+			(project "powersupplies_kicadproject"
 				(path "/d2bb73ea-a6bc-4588-b3f4-545ae2e25abc/b247aa19-c6db-40d4-9578-4858bd0a46c8"
 					(reference "#PWR02")
@@
 		)
 		(instances
-			(project "Eurocard_48pin_AMO_Blank"
+			(project "powersupplies_kicadproject"
 				(path "/d2bb73ea-a6bc-4588-b3f4-545ae2e25abc/b247aa19-c6db-40d4-9578-4858bd0a46c8"
 					(reference "#PWR011")
@@
 		)
 		(instances
-			(project "Eurocard_48pin_AMO_Blank"
+			(project "powersupplies_kicadproject"
 				(path "/d2bb73ea-a6bc-4588-b3f4-545ae2e25abc/b247aa19-c6db-40d4-9578-4858bd0a46c8"
 					(reference "U1")
@@
 		)
 		(instances
-			(project "Eurocard_48pin_AMO_Blank"
+			(project "powersupplies_kicadproject"
 				(path "/d2bb73ea-a6bc-4588-b3f4-545ae2e25abc/b247aa19-c6db-40d4-9578-4858bd0a46c8"
 					(reference "#PWR06")
@@
 		)
 		(instances
-			(project "Eurocard_48pin_AMO_Blank"
+			(project "powersupplies_kicadproject"
 				(path "/d2bb73ea-a6bc-4588-b3f4-545ae2e25abc/b247aa19-c6db-40d4-9578-4858bd0a46c8"
 					(reference "U1")
@@
 		)
 		(instances
-			(project "Eurocard_48pin_AMO_Blank"
+			(project "powersupplies_kicadproject"
 				(path "/d2bb73ea-a6bc-4588-b3f4-545ae2e25abc/b247aa19-c6db-40d4-9578-4858bd0a46c8"
 					(reference "#PWR01")
@@
 		)
 		(instances
-			(project "Eurocard_48pin_AMO_Blank"
+			(project "powersupplies_kicadproject"
 				(path "/d2bb73ea-a6bc-4588-b3f4-545ae2e25abc/b247aa19-c6db-40d4-9578-4858bd0a46c8"
 					(reference "U1")
@@
 		)
 		(instances
-			(project "Eurocard_48pin_AMO_Blank"
+			(project "powersupplies_kicadproject"
 				(path "/d2bb73ea-a6bc-4588-b3f4-545ae2e25abc/b247aa19-c6db-40d4-9578-4858bd0a46c8"
 					(reference "#PWR012")
@@
 		)
 		(instances
-			(project "Eurocard_48pin_AMO_Blank"
+			(project "powersupplies_kicadproject"
 				(path "/d2bb73ea-a6bc-4588-b3f4-545ae2e25abc/b247aa19-c6db-40d4-9578-4858bd0a46c8"
 					(reference "#PWR010")
@@
 		)
 		(instances
-			(project "Eurocard_48pin_AMO_Blank"
+			(project "powersupplies_kicadproject"
 				(path "/d2bb73ea-a6bc-4588-b3f4-545ae2e25abc/b247aa19-c6db-40d4-9578-4858bd0a46c8"
 					(reference "U1")
